Commit message: introduce ee_link

File: ar_moveit_config/srdf/ar_gripper_macro.srdf.xacro (robot description, xacro)
@@ -17,9 +17,9 @@
     </group_state>
     <group_state name="closed" group="ar_gripper">
-      <joint name="gripper_jaw1_joint" value="0" />
+      <joint name="gripper_jaw1_joint" value="-0.01" />
     </group_state>
     <disable_collisions link1="gripper_base_link" link2="gripper_jaw1_link" reason="Adjacent" />
     <disable_collisions link1="gripper_base_link" link2="gripper_jaw2_link" reason="Adjacent" />
-    <disable_collisions link1="gripper_jaw1_link" link2="gripper_jaw2_link" reason="Adjacent" />
+    <disable_collisions link1="gripper_jaw1_link" link2="gripper_jaw2_link" reason="Default" />
     <disable_collisions link1="link_6" link2="gripper_base_link" reason="Adjacent" />
   </xacro:macro>

Commit message: tweak gripper closed position

File: ar_moveit_config/srdf/ar_gripper_macro.srdf.xacro (robot description, xacro)
@@ -17,5 +17,5 @@
     </group_state>
     <group_state name="closed" group="ar_gripper">
-      <joint name="gripper_jaw1_joint" value="-0.01" />
+      <joint name="gripper_jaw1_joint" value="-0.001" />
     </group_state>
     <disable_collisions link1="gripper_base_link" link2="gripper_jaw1_link" reason="Adjacent" />
