Commit message: nice! track can be unset for demo. (notrack)controllers.yaml should still be done

File: ar_moveit_config/srdf/ar_macro.srdf.xacro (robot description, xacro)
@@ -7,4 +7,5 @@
 <robot xmlns:xacro="http://wiki.ros.org/xacro">
   <xacro:macro name="ar_srdf">
+    <xacro:arg name="include_track" default="True" />
     <group name="ar_manipulator">
       <joint name="joint_1" />
@@ -16,23 +17,25 @@
       <joint name="ee_joint" />
     </group>
-    <group name="ar_track_manipulator">
-      <joint name="joint_1" />
-      <joint name="joint_2" />
-      <joint name="joint_3" />
-      <joint name="joint_4" />
-      <joint name="joint_5" />
-      <joint name="joint_6" />
-      <joint name="ee_joint" />
-      <joint name="linear_slider_joint" />
-    </group>
-    <group_state name="home" group="ar_track_manipulator">
-      <joint name="joint_1" value="0" />
-      <joint name="joint_2" value="0" />
-      <joint name="joint_3" value="0" />
-      <joint name="joint_4" value="0" />
-      <joint name="joint_5" value="0" />
-      <joint name="joint_6" value="0" />
-      <joint name="linear_slider_joint" value="0" />
-    </group_state>
+    <xacro:if value="$(arg include_track)">
+      <group name="ar_track_manipulator">
+        <joint name="joint_1" />
+        <joint name="joint_2" />
+        <joint name="joint_3" />
+        <joint name="joint_4" />
+        <joint name="joint_5" />
+        <joint name="joint_6" />
+        <joint name="ee_joint" />
+        <joint name="linear_slider_joint" />
+      </group>
+      <group_state name="home" group="ar_track_manipulator">
+        <joint name="joint_1" value="0" />
+        <joint name="joint_2" value="0" />
+        <joint name="joint_3" value="0" />
+        <joint name="joint_4" value="0" />
+        <joint name="joint_5" value="0" />
+        <joint name="joint_6" value="0" />
+        <joint name="linear_slider_joint" value="0" />
+      </group_state>
+    </xacro:if>
     <group_state name="home" group="ar_manipulator">
       <joint name="joint_1" value="0" />
