Commit message: demo broken and plate too thick otherwise nice

File: ar_description/urdf/ar_track_macro.xacro (robot description, xacro)
@@ -39,5 +39,5 @@
       <origin xyz="0 0 ${robot_parameters['linear_track_height']}" rpy="0 0 0" />
       <axis xyz="1 0 0" />
-      <limit lower="${-0.1-robot_parameters['linear_track_length']/2+0.15/2}"
+      <limit lower="${-robot_parameters['linear_track_length']/2+0.15/2}"
         upper="${robot_parameters['linear_track_length']/2-0.15/2}" effort="100" velocity="0.5" />
     </joint>
