Commit message: so great and so beautiful !

File: ar_description/urdf/ar.urdf.xacro (robot description, xacro)
@@ -1,33 +1,29 @@
 <?xml version="1.0"?>
 <robot xmlns:xacro="http://wiki.ros.org/xacro" name="$(arg ar_model)">
-  <xacro:arg name="include_gripper" default="true" />
-  <xacro:arg name="include_track" default="true" />
+  <xacro:arg name="include_gripper" default="True" />
+  <xacro:arg name="include_track" default="True" />
   <xacro:include filename="$(find ar_description)/urdf/ar_macro.xacro" />
-  <!-- clean this up -->
   <xacro:property name="robot_parameters_file"
     value="$(find ar_description)/config/$(arg ar_model).yaml" />
   <xacro:property name="robot_parameters" value="${xacro.load_yaml(robot_parameters_file)}" />
-  <!-- clean this up -->
   <link name="world" />
+  <xacro:property name="ar_robot_parent" value="world" />
+  <xacro:property name="ar_robot_origin_xyz" value="0 0 0" />
   <xacro:if value="$(arg include_track)">
-    <xacro:include filename="$(find ar_description)/urdf/ar_track.xacro" />
+    <xacro:include filename="$(find ar_description)/urdf/ar_track_macro.xacro" />
     <xacro:ar_track
       parent="world"
-      robot_parameters_file="$(find ar_description)/config/$(arg ar_model).yaml">
+      robot_parameters_file="${robot_parameters_file}">
       <origin xyz="0 0 0" rpy="0 0 0" />
     </xacro:ar_track>
-    <xacro:ar_robot
-      parent="linear_slider_link"
-      robot_parameters_file="$(find ar_description)/config/$(arg ar_model).yaml">
-      <origin xyz="0 0 ${robot_parameters['linear_plate_height']}" rpy="0 0 0" />
-    </xacro:ar_robot>
+    <xacro:property name="ar_robot_parent" value="linear_slider_link" />
+    <xacro:property name="ar_robot_origin_xyz"
+      value="0 0 ${robot_parameters['linear_plate_height']}" />
   </xacro:if>
-  <xacro:unless value="$(arg include_track)">
-    <xacro:ar_robot
-      parent="world"
-      robot_parameters_file="$(find ar_description)/config/$(arg ar_model).yaml">
-      <origin xyz="0 0 0" rpy="0 0 0" />
-    </xacro:ar_robot>
-  </xacro:unless>
+  <xacro:ar_robot
+    parent="${ar_robot_parent}"
+    robot_parameters_file="${robot_parameters_file}">
+    <origin xyz="${ar_robot_origin_xyz}" rpy="0 0 0" />
+  </xacro:ar_robot>
   <xacro:if value="$(arg include_gripper)">
     <xacro:include filename="$(find ar_description)/urdf/ar_gripper_macro.xacro" />

File: ar_description/urdf/ar_gazebo.urdf.xacro (robot description, xacro)
@@ -2,35 +2,31 @@
 <robot xmlns:xacro="http://wiki.ros.org/xacro" name="$(arg ar_model)">
   <xacro:arg name="simulation_controllers" default="" />
-  <xacro:arg name="include_gripper" default="true" />
-  <xacro:arg name="include_track" default="true" />
+  <xacro:arg name="include_gripper" default="True" />
+  <xacro:arg name="include_track" default="True" />
   <xacro:include filename="$(find ar_description)/urdf/ar_macro.xacro" />
   <xacro:include filename="$(find ar_description)/urdf/ar.ros2_control.xacro" />
   <xacro:include filename="$(find ar_description)/urdf/ar_gripper.ros2_control.xacro" />
-  <!-- clean this up -->
   <xacro:property name="robot_parameters_file"
     value="$(find ar_description)/config/$(arg ar_model).yaml" />
   <xacro:property name="robot_parameters" value="${xacro.load_yaml(robot_parameters_file)}" />
-  <!-- clean this up -->
   <link name="world" />
+  <xacro:property name="ar_robot_parent" value="world" />
+  <xacro:property name="ar_robot_origin_xyz" value="0 0 0" />
   <xacro:if value="$(arg include_track)">
-    <xacro:include filename="$(find ar_description)/urdf/ar_track.xacro" />
+    <xacro:include filename="$(find ar_description)/urdf/ar_track_macro.xacro" />
     <xacro:ar_track
       parent="world"
-      robot_parameters_file="$(find ar_description)/config/$(arg ar_model).yaml">
+      robot_parameters_file="${robot_parameters_file}">
       <origin xyz="0 0 0" rpy="0 0 0" />
     </xacro:ar_track>
-    <xacro:ar_robot
-      parent="linear_slider_link"
-      robot_parameters_file="$(find ar_description)/config/$(arg ar_model).yaml">
-      <origin xyz="0 0 ${robot_parameters['linear_plate_height']}" rpy="0 0 0" />
-    </xacro:ar_robot>
+    <xacro:property name="ar_robot_parent" value="linear_slider_link" />
+    <xacro:property name="ar_robot_origin_xyz"
+      value="0 0 ${robot_parameters['linear_plate_height']}" />
   </xacro:if>
-  <xacro:unless value="$(arg include_track)">
-    <xacro:ar_robot
-      parent="world"
-      robot_parameters_file="$(find ar_description)/config/$(arg ar_model).yaml">
-      <origin xyz="0 0 0" rpy="0 0 0" />
-    </xacro:ar_robot>
-  </xacro:unless>
+  <xacro:ar_robot
+    parent="${ar_robot_parent}"
+    robot_parameters_file="${robot_parameters_file}">
+    <origin xyz="${ar_robot_origin_xyz}" rpy="0 0 0" />
+  </xacro:ar_robot>
   <xacro:if value="$(arg include_gripper)">
     <xacro:include filename="$(find ar_description)/urdf/ar_gripper_macro.xacro" />

File: ar_hardware_interface/urdf/ar.urdf.xacro (robot description, xacro)
@@ -1,16 +1,31 @@
 <?xml version="1.0"?>
 <robot xmlns:xacro="http://wiki.ros.org/xacro" name="$(arg ar_model)">
-  <xacro:arg name="serial_port" default="/dev/ttyACM0"/>
-  <xacro:arg name="arduino_serial_port" default="/dev/ttyUSB0"/>
-  <xacro:arg name="calibrate" default="True"/>
-  <xacro:arg name="include_gripper" default="true"/>
-  <xacro:include filename="$(find ar_description)/urdf/ar_macro.xacro"/>
-  <xacro:include filename="$(find ar_description)/urdf/ar.ros2_control.xacro"/>
-  <link name="world" />
+  <xacro:arg name="serial_port" default="/dev/ttyACM0" />
+  <xacro:arg name="arduino_serial_port" default="/dev/ttyUSB0" />
+  <xacro:arg name="calibrate" default="True" />
+  <xacro:arg name="include_gripper" default="True" />
+  <xacro:arg name="include_track" default="True" />
+  <xacro:include filename="$(find ar_description)/urdf/ar_macro.xacro" />
+  <xacro:include filename="$(find ar_description)/urdf/ar.ros2_control.xacro" />
+  <xacro:property name="robot_parameters_file"
+    value="$(find ar_description)/config/$(arg ar_model).yaml" />
+  <xacro:property name="robot_parameters" value="${xacro.load_yaml(robot_parameters_file)}" />
+  <xacro:property name="ar_robot_parent" value="world" />
+  <xacro:property name="ar_robot_origin_xyz" value="0 0 0" />
+  <xacro:if value="$(arg include_track)">
+    <xacro:include filename="$(find ar_description)/urdf/ar_track_macro.xacro" />
+    <xacro:ar_track
+      parent="world"
+      robot_parameters_file="${robot_parameters_file}">
+      <origin xyz="0 0 0" rpy="0 0 0" />
+    </xacro:ar_track>
+    <xacro:property name="ar_robot_parent" value="linear_slider_link" />
+    <xacro:property name="ar_robot_origin_xyz"
+      value="0 0 ${robot_parameters['linear_plate_height']}" />
+  </xacro:if>
   <xacro:ar_robot
-    parent="world"
-    robot_parameters_file="$(find ar_description)/config/$(arg ar_model).yaml"
-  >
-    <origin xyz="0 0 0" rpy="0 0 0" />
+    parent="${ar_robot_parent}"
+    robot_parameters_file="${robot_parameters_file}">
+    <origin xyz="${ar_robot_origin_xyz" rpy="0 0 0" />
   </xacro:ar_robot>
   <xacro:ar_ros2_control
@@ -22,6 +37,6 @@
   />
   <xacro:if value="$(arg include_gripper)">
-    <xacro:include filename="$(find ar_description)/urdf/ar_gripper_macro.xacro"/>
-    <xacro:include filename="$(find ar_description)/urdf/ar_gripper.ros2_control.xacro"/>
+    <xacro:include filename="$(find ar_description)/urdf/ar_gripper_macro.xacro" />
+    <xacro:include filename="$(find ar_description)/urdf/ar_gripper.ros2_control.xacro" />
     <xacro:ar_gripper parent="ee_link" />
     <xacro:ar_gripper_ros2_control

File: ar_moveit_config/srdf/ar.srdf.xacro (robot description, xacro)
@@ -1,6 +1,6 @@
 <?xml version="1.0" encoding="UTF-8"?>
 <robot xmlns:xacro="http://wiki.ros.org/xacro" name="$(arg name)">
-  <xacro:arg name="include_gripper" default="true" />
-  <xacro:arg name="include_track" default="true" />
+  <xacro:arg name="include_gripper" default="True" />
+  <xacro:arg name="include_track" default="True" />
   <xacro:if value="$(arg include_track)">
     <xacro:include filename="$(find ar_moveit_config)/srdf/ar_track_macro.srdf.xacro" />

File: ar_moveit_config/srdf/ar_macro.srdf.xacro (robot description, xacro)
@@ -16,4 +16,23 @@
       <joint name="ee_joint" />
     </group>
+    <group name="ar_track_manipulator">
+      <joint name="joint_1" />
+      <joint name="joint_2" />
+      <joint name="joint_3" />
+      <joint name="joint_4" />
+      <joint name="joint_5" />
+      <joint name="joint_6" />
+      <joint name="ee_joint" />
+      <joint name="linear_slider_joint" />
+    </group>
+    <group_state name="home" group="ar_track_manipulator">
+      <joint name="joint_1" value="0" />
+      <joint name="joint_2" value="0" />
+      <joint name="joint_3" value="0" />
+      <joint name="joint_4" value="0" />
+      <joint name="joint_5" value="0" />
+      <joint name="joint_6" value="0" />
+      <joint name="linear_slider_joint" value="0" />
+    </group_state>
     <group_state name="home" group="ar_manipulator">
       <joint name="joint_1" value="0" />

File: ar_moveit_config/urdf/fake_ar.urdf.xacro (robot description, xacro)
@@ -1,8 +1,8 @@
 <?xml version="1.0"?>
 <robot xmlns:xacro="http://wiki.ros.org/xacro" name="$(arg ar_model)">
-  <xacro:include filename="$(find ar_description)/urdf/ar_macro.xacro"/>
-  <xacro:include filename="$(find ar_description)/urdf/ar_gripper_macro.xacro"/>
-  <xacro:include filename="$(find ar_description)/urdf/ar.ros2_control.xacro"/>
-  <xacro:include filename="$(find ar_description)/urdf/ar_gripper.ros2_control.xacro"/>
+  <xacro:include filename="$(find ar_description)/urdf/ar_macro.xacro" />
+  <xacro:include filename="$(find ar_description)/urdf/ar_gripper_macro.xacro" />
+  <xacro:include filename="$(find ar_description)/urdf/ar.ros2_control.xacro" />
+  <xacro:include filename="$(find ar_description)/urdf/ar_gripper.ros2_control.xacro" />
   <link name="world" />
   <xacro:ar_robot

Commit message: Let's try to simplify ar_gazebo.urdf

File: ar_description/urdf/ar.urdf.xacro (robot description, xacro)
@@ -30,3 +30,9 @@
     <xacro:ar_gripper parent="ee_link" />
   </xacro:if>
+  <xacro:include filename="$(find ar_description)/urdf/ar_camera_macro.xacro" />
+  <xacro:ar_camera
+    parent="base_link"
+    robot_parameters_file="${robot_parameters_file}">
+    <origin xyz="0 0 0" rpy="0 0 0" />
+  </xacro:ar_camera>
 </robot>

File: ar_description/urdf/ar_gazebo.urdf.xacro (robot description, xacro)
@@ -33,4 +33,10 @@
     <xacro:ar_gripper parent="ee_link" />
   </xacro:if>
+  <xacro:include filename="$(find ar_description)/urdf/ar_camera_macro.xacro" />
+  <xacro:ar_camera
+    parent="base_link"
+    robot_parameters_file="${robot_parameters_file}">
+    <origin xyz="0 0 0" rpy="0 0 0" />
+  </xacro:ar_camera>
   <xacro:ar_ros2_control
     name="ARGazeboSystem"

File: ar_description/urdf/ar_track_macro.xacro (robot description, xacro)
@@ -5,11 +5,35 @@
   robot_parameters_file">
     <xacro:property name="robot_parameters" value="${xacro.load_yaml(robot_parameters_file)}" />
-    <xacro:property name="plate_width" value="${robot_parameters['linear_plate_width']}" />
-    <xacro:property name="plate_length" value="${robot_parameters['linear_plate_length']}" />
-    <xacro:property name="plate_height" value="${robot_parameters['linear_plate_height']}" />
-    <xacro:property name="track_width" value="${robot_parameters['linear_track_width']}" />
-    <xacro:property name="track_length" value="${robot_parameters['linear_track_length']}" />
-    <xacro:property name="track_height" value="${robot_parameters['linear_track_height']}" />
-    <joint name="linear_base_joint" type="fixed">
+    <xacro:property
+      name="plate_width" value="${robot_parameters['linear_plate_width']}" />
+    <xacro:property
+      name="plate_length" value="${robot_parameters['linear_plate_length']}" />
+    <xacro:property
+      name="plate_height" value="${robot_parameters['linear_plate_height']}" />
+    <xacro:property
+      name="track_width" value="${robot_parameters['linear_track_width']}" />
+    <xacro:property
+      name="track_length" value="${robot_parameters['linear_track_length']}" />
+    <xacro:property
+      name="track_height" value="${robot_parameters['linear_track_height']}" />
+    <xacro:property
+      name="bearing_spacer" value="${robot_parameters['linear_bearing_spacer']}" />
+    <xacro:macro
+      name="block_corner" params="x y">
+      <visual>
+        <origin
+          xyz="${x*(plate_width-bearing_spacer)/2} ${y*(plate_length-bearing_spacer)/2} ${-plate_height / 2}"
+          rpy="0 0 0" />
+        <geometry>
+          <mesh
+            filename="file://$(find ar_description)/meshes/${robot_parameters['mesh_dir']}/track_bearing.stl" />
+        </geometry>
+      </visual>
+      <material name="">
+        <color rgba="1 1 0 1" />
+      </material>
+    </xacro:macro>
+    <joint name="linear_base_joint"
+      type="fixed">
       <xacro:insert_block name="origin" />
       <parent link="${parent}" />
@@ -24,5 +48,5 @@
       <visual>
         <origin
-          xyz="0 ${-track_width/2+0.03/2} ${track_height / 2}"
+          xyz="0 ${(-track_width+bearing_spacer)/2} ${track_height / 2}"
           rpy="0 0 0" />
         <geometry>
@@ -36,5 +60,5 @@
       <visual>
         <origin
-          xyz="0 ${track_width/2-0.03/2} ${track_height / 2}"
+          xyz="0 ${(track_width-bearing_spacer)/2} ${track_height / 2}"
           rpy="0 0 0" />
         <geometry>
@@ -54,5 +78,9 @@
       </collision>
     </link>
-    <joint name="linear_slider_joint" type="prismatic">
+    <gazebo reference="linear_slider_link">
+      <material>Gazebo/Grey</material>
+    </gazebo>
+    <joint
+      name="linear_slider_joint" type="prismatic">
       <parent link="linear_base_link" />
       <child link="linear_slider_link" />
@@ -80,16 +108,8 @@
         </material>
       </visual>
-      <visual>
-        <origin
-          xyz="${plate_width/2} ${plate_length/2} ${-plate_height / 2}"
-          rpy="0 0 0" />
-        <geometry>
-          <mesh
-            filename="file://$(find ar_description)/meshes/${robot_parameters['mesh_dir']}/track_bearing.stl" />
-        </geometry>
-        <material name="">
-          <color rgba="1 1 0 1" />
-        </material>
-      </visual>
+      <xacro:block_corner x="1" y="1" />
+      <xacro:block_corner x="1" y="-1" />
+      <xacro:block_corner x="-1" y="1" />
+      <xacro:block_corner x="-1" y="-1" />
       <collision>
         <origin xyz="0 0 ${plate_height / 2}" rpy="0 0 0" />

Commit message: Camera simulation is up and running

File: ar_description/urdf/ar.urdf.xacro (robot description, xacro)
@@ -3,15 +3,16 @@
   <xacro:arg name="include_gripper" default="True" />
   <xacro:arg name="include_track" default="True" />
+  <xacro:arg name="include_camera" default="True" />
   <xacro:include filename="$(find ar_description)/urdf/ar_macro.xacro" />
   <xacro:property name="robot_parameters_file"
     value="$(find ar_description)/config/$(arg ar_model).yaml" />
   <xacro:property name="robot_parameters" value="${xacro.load_yaml(robot_parameters_file)}" />
-  <link name="world" />
-  <xacro:property name="ar_robot_parent" value="world" />
+  <link name="aworld" /> <!-- not locked to WORLD, so then we can link camera to this .. -->
+  <xacro:property name="ar_robot_parent" value="aworld" />
   <xacro:property name="ar_robot_origin_xyz" value="0 0 0" />
   <xacro:if value="$(arg include_track)">
     <xacro:include filename="$(find ar_description)/urdf/ar_track_macro.xacro" />
     <xacro:ar_track
-      parent="world"
+      parent="${ar_robot_parent}"
       robot_parameters_file="${robot_parameters_file}">
       <origin xyz="0 0 0" rpy="0 0 0" />
@@ -30,9 +31,11 @@
     <xacro:ar_gripper parent="ee_link" />
   </xacro:if>
-  <xacro:include filename="$(find ar_description)/urdf/ar_camera_macro.xacro" />
-  <xacro:ar_camera
-    parent="base_link"
-    robot_parameters_file="${robot_parameters_file}">
-    <origin xyz="0 0 0" rpy="0 0 0" />
-  </xacro:ar_camera>
+  <xacro:if value="$(arg include_track)">
+    <xacro:include filename="$(find ar_description)/urdf/ar_camera_macro.xacro" />
+    <xacro:ar_camera
+      parent="${ar_robot_parent}"
+      robot_parameters_file="${robot_parameters_file}">
+      <origin xyz="0 -0.75 1" rpy="0 ${pi/2} ${pi/2}" />
+    </xacro:ar_camera>
+  </xacro:if>
 </robot>

File: ar_description/urdf/ar_camera_macro.xacro (robot description, xacro)
@@ -42,4 +42,9 @@
         <plugin name="camera_controller" filename="libgazebo_ros_camera.so">
           <frame_name>camera_link_optical</frame_name>
+          <alwaysOn>true</alwaysOn>
+          <updateRate>0.0</updateRate>
+          <cameraName>camera1</cameraName>
+          <imageTopicName>image_raw</imageTopicName>
+          <cameraInfoTopicName>camera_info</cameraInfoTopicName>
         </plugin>
       </sensor>

File: ar_description/urdf/ar_gazebo.urdf.xacro (robot description, xacro)
@@ -4,39 +4,10 @@
   <xacro:arg name="include_gripper" default="True" />
   <xacro:arg name="include_track" default="True" />
-  <xacro:include filename="$(find ar_description)/urdf/ar_macro.xacro" />
+  <xacro:arg name="include_camera" default="True" />
+  <xacro:include filename="$(find ar_description)/urdf/ar.urdf.xacro" />
+  <!--<xacro:include
+  filename="$(find ar_description)/urdf/ar_macro.xacro" />-->
   <xacro:include filename="$(find ar_description)/urdf/ar.ros2_control.xacro" />
   <xacro:include filename="$(find ar_description)/urdf/ar_gripper.ros2_control.xacro" />
-  <xacro:property name="robot_parameters_file"
-    value="$(find ar_description)/config/$(arg ar_model).yaml" />
-  <xacro:property name="robot_parameters" value="${xacro.load_yaml(robot_parameters_file)}" />
-  <link name="world" /> <!-- rename to have robot "free"-->
-  <xacro:property name="ar_robot_parent" value="world" />
-  <xacro:property name="ar_robot_origin_xyz" value="0 0 0" />
-  <xacro:if value="$(arg include_track)">
-    <xacro:include filename="$(find ar_description)/urdf/ar_track_macro.xacro" />
-    <xacro:ar_track
-      parent="world"
-      robot_parameters_file="${robot_parameters_file}">
-      <origin xyz="0 0 0" rpy="0 0 0" />
-    </xacro:ar_track>
-    <xacro:property name="ar_robot_parent" value="linear_slider_link" />
-    <xacro:property name="ar_robot_origin_xyz"
-      value="0 0 ${robot_parameters['linear_plate_height']}" />
-  </xacro:if>
-  <xacro:ar_robot
-    parent="${ar_robot_parent}"
-    robot_parameters_file="${robot_parameters_file}">
-    <origin xyz="${ar_robot_origin_xyz}" rpy="0 0 0" />
-  </xacro:ar_robot>
-  <xacro:if value="$(arg include_gripper)">
-    <xacro:include filename="$(find ar_description)/urdf/ar_gripper_macro.xacro" />
-    <xacro:ar_gripper parent="ee_link" />
-  </xacro:if>
-  <xacro:include filename="$(find ar_description)/urdf/ar_camera_macro.xacro" />
-  <xacro:ar_camera
-    parent="base_link"
-    robot_parameters_file="${robot_parameters_file}">
-    <origin xyz="0 0 0" rpy="0 0 0" />
-  </xacro:ar_camera>
   <xacro:ar_ros2_control
     name="ARGazeboSystem"

Commit message: old working

File: ar_description/urdf/ar.urdf.xacro (robot description, xacro)
@@ -3,11 +3,11 @@
   <xacro:arg name="include_gripper" default="True" />
   <xacro:arg name="include_track" default="True" />
-  <xacro:arg name="include_camera" default="True" />
+  <xacro:arg name="include_camera" default="False" />
   <xacro:include filename="$(find ar_description)/urdf/ar_macro.xacro" />
   <xacro:property name="robot_parameters_file"
     value="$(find ar_description)/config/$(arg ar_model).yaml" />
   <xacro:property name="robot_parameters" value="${xacro.load_yaml(robot_parameters_file)}" />
-  <link name="aworld" /> <!-- not locked to WORLD, so then we can link camera to this .. -->
-  <xacro:property name="ar_robot_parent" value="aworld" />
+  <link name="world" /> <!-- not locked to WORLD, so then we can link camera to this .. -->
+  <xacro:property name="ar_robot_parent" value="world" />
   <xacro:property name="ar_robot_origin_xyz" value="0 0 0" />
   <xacro:if value="$(arg include_track)">
@@ -31,5 +31,5 @@
     <xacro:ar_gripper parent="ee_link" />
   </xacro:if>
-  <xacro:if value="$(arg include_track)">
+  <xacro:if value="$(arg include_camera)">
     <xacro:include filename="$(find ar_description)/urdf/ar_camera_macro.xacro" />
     <xacro:ar_camera

File: ar_hardware_interface/urdf/ar.urdf.xacro (robot description, xacro)
@@ -6,4 +6,5 @@
   <xacro:arg name="include_gripper" default="True" />
   <xacro:arg name="include_track" default="True" />
+  <xacro:arg name="include_camera" default="False" />
   <xacro:include filename="$(find ar_description)/urdf/ar_macro.xacro" />
   <xacro:include filename="$(find ar_description)/urdf/ar.ros2_control.xacro" />
@@ -11,4 +12,5 @@
     value="$(find ar_description)/config/$(arg ar_model).yaml" />
   <xacro:property name="robot_parameters" value="${xacro.load_yaml(robot_parameters_file)}" />
+  <link name="world" /> <!-- not locked to WORLD, so then we can link camera to this .. -->
   <xacro:property name="ar_robot_parent" value="world" />
   <xacro:property name="ar_robot_origin_xyz" value="0 0 0" />
@@ -16,5 +18,5 @@
     <xacro:include filename="$(find ar_description)/urdf/ar_track_macro.xacro" />
     <xacro:ar_track
-      parent="world"
+      parent="${ar_robot_parent}"
       robot_parameters_file="${robot_parameters_file}">
       <origin xyz="0 0 0" rpy="0 0 0" />
@@ -27,5 +29,5 @@
     parent="${ar_robot_parent}"
     robot_parameters_file="${robot_parameters_file}">
-    <origin xyz="${ar_robot_origin_xyz" rpy="0 0 0" />
+    <origin xyz="${ar_robot_origin_xyz}" rpy="0 0 0" />
   </xacro:ar_robot>
   <xacro:ar_ros2_control
@@ -46,3 +48,11 @@
     />
   </xacro:if>
+  <xacro:if value="$(arg include_camera)">
+    <xacro:include filename="$(find ar_description)/urdf/ar_camera_macro.xacro" />
+    <xacro:ar_camera
+      parent="${ar_robot_parent}"
+      robot_parameters_file="${robot_parameters_file}">
+      <origin xyz="0 -0.75 1" rpy="0 ${pi/2} ${pi/2}" />
+    </xacro:ar_camera>
+  </xacro:if>
 </robot>
