Commit message: Personal MK3-changes

File: ar_description/urdf/ar.ros2_control.xacro (robot description, xacro)
@@ -48,6 +48,6 @@
       <joint name="joint_4">
         <command_interface name="position">
-          <param name="min">{-165*pi/180}</param>
-          <param name="max">{165*pi/180}</param>
+          <param name="min">{-180*pi/180}</param>
+          <param name="max">{180*pi/180}</param>
         </command_interface>
         <state_interface name="position">
@@ -68,6 +68,6 @@
       <joint name="joint_6">
         <command_interface name="position">
-          <param name="min">{-155*pi/180}</param>
-          <param name="max">{155*pi/180}</param>
+          <param name="min">{-180*pi/180}</param>
+          <param name="max">{180*pi/180}</param>
         </command_interface>
         <state_interface name="position">

File: ar_moveit_config/srdf/ar_gripper_macro.srdf.xacro (robot description, xacro)
@@ -1,3 +1,3 @@
-<?xml version="1.0" ?>
+<?xml version="1.0"?>
 <!--This does not replace URDF, and is not an extension of URDF.
     This is a format for representing semantic information about the robot structure.
@@ -14,5 +14,5 @@
     </group>
     <group_state name="open" group="ar_gripper">
-      <joint name="gripper_jaw1_joint" value="-0.012" />
+      <joint name="gripper_jaw1_joint" value="-0.027" />
     </group_state>
     <group_state name="closed" group="ar_gripper">

File: ar_moveit_config/srdf/ar_macro.srdf.xacro (robot description, xacro)
@@ -1,3 +1,3 @@
-<?xml version="1.0" ?>
+<?xml version="1.0"?>
 <!--This does not replace URDF, and is not an extension of URDF.
     This is a format for representing semantic information about the robot structure.
@@ -13,5 +13,5 @@
       <joint name="joint_5" />
       <joint name="joint_6" />
-      <joint name="ee_joint"/>
+      <joint name="ee_joint" />
     </group>
     <group_state name="home" group="ar_manipulator">
@@ -25,6 +25,6 @@
     <group_state name="upright" group="ar_manipulator">
       <joint name="joint_1" value="0" />
-      <joint name="joint_2" value="-0.087" />
-      <joint name="joint_3" value="-1.34" />
+      <joint name="joint_2" value="0" />
+      <joint name="joint_3" value="-1.55" />
       <joint name="joint_4" value="0" />
       <joint name="joint_5" value="0" />
