Commit message: linear track
stable in gazebo

nope..not stable

testing

promising

yes! next control

File: ar_description/urdf/ar.ros2_control.xacro (robot description, xacro)
@@ -1,5 +1,6 @@
 <?xml version="1.0"?>
 <robot xmlns:xacro="http://www.ros.org/wiki/xacro">
-  <xacro:macro name="ar_ros2_control" params="
+  <xacro:macro name="ar_ros2_control"
+    params="
     name
     plugin_name
@@ -9,5 +10,5 @@
   ">
     <xacro:property name="joint_offset_parameters"
-      value="${xacro.load_yaml(joint_offset_parameters_file)}"/>
+      value="${xacro.load_yaml(joint_offset_parameters_file)}" />
     <ros2_control name="${name}" type="system">
       <hardware>
@@ -16,4 +17,14 @@
         <param name="calibrate">${calibrate}</param>
       </hardware>
+      <joint name="linear_slider_joint">
+        <command_interface name="position">
+          <param name="min">{-0.6/2+0.15/2}</param>
+          <param name="max">{0.6/2-0.15/2}</param>
+        </command_interface>
+        <state_interface name="position">
+          <param name="initial_value">0.0</param>
+        </state_interface>
+        <param name="position_offset">${joint_offset_parameters['linear_track']}</param>
+      </joint>
       <joint name="joint_1">
         <command_interface name="position">

File: ar_description/urdf/ar.urdf.xacro (robot description, xacro)
@@ -1,15 +1,35 @@
 <?xml version="1.0"?>
 <robot xmlns:xacro="http://wiki.ros.org/xacro" name="$(arg ar_model)">
-  <xacro:arg name="include_gripper" default="true"/>
-  <xacro:include filename="$(find ar_description)/urdf/ar_macro.xacro"/>
+  <xacro:arg name="include_gripper" default="true" />
+  <xacro:arg name="include_track" default="true" />
+  <xacro:include filename="$(find ar_description)/urdf/ar_macro.xacro" />
+  <!-- clean this up -->
+  <xacro:property name="robot_parameters_file"
+    value="$(find ar_description)/config/$(arg ar_model).yaml" />
+  <xacro:property name="robot_parameters" value="${xacro.load_yaml(robot_parameters_file)}" />
+  <!-- clean this up -->
   <link name="world" />
-  <xacro:ar_robot
-    parent="world"
-    robot_parameters_file="$(find ar_description)/config/$(arg ar_model).yaml"
-  >
-    <origin xyz="0 0 0" rpy="0 0 0" />
-  </xacro:ar_robot>
+  <xacro:if value="$(arg include_track)">
+    <xacro:include filename="$(find ar_description)/urdf/ar_track.xacro" />
+    <xacro:ar_track
+      parent="world"
+      robot_parameters_file="$(find ar_description)/config/$(arg ar_model).yaml">
+      <origin xyz="0 0 0" rpy="0 0 0" />
+    </xacro:ar_track>
+    <xacro:ar_robot
+      parent="linear_slider_link"
+      robot_parameters_file="$(find ar_description)/config/$(arg ar_model).yaml">
+      <origin xyz="0 0 ${robot_parameters['linear_plate_height']}" rpy="0 0 0" />
+    </xacro:ar_robot>
+  </xacro:if>
+  <xacro:unless value="$(arg include_track)">
+    <xacro:ar_robot
+      parent="world"
+      robot_parameters_file="$(find ar_description)/config/$(arg ar_model).yaml">
+      <origin xyz="0 0 0" rpy="0 0 0" />
+    </xacro:ar_robot>
+  </xacro:unless>
   <xacro:if value="$(arg include_gripper)">
-    <xacro:include filename="$(find ar_description)/urdf/ar_gripper_macro.xacro"/>
+    <xacro:include filename="$(find ar_description)/urdf/ar_gripper_macro.xacro" />
     <xacro:ar_gripper parent="ee_link" />
   </xacro:if>

File: ar_description/urdf/ar_gazebo.urdf.xacro (robot description, xacro)
@@ -1,17 +1,40 @@
 <?xml version="1.0"?>
 <robot xmlns:xacro="http://wiki.ros.org/xacro" name="$(arg ar_model)">
+  <xacro:arg name="simulation_controllers" default="" />
+  <xacro:arg name="include_gripper" default="true" />
+  <xacro:arg name="include_track" default="true" />
   <xacro:include filename="$(find ar_description)/urdf/ar_macro.xacro" />
-  <xacro:include filename="$(find ar_description)/urdf/ar_gripper_macro.xacro" />
   <xacro:include filename="$(find ar_description)/urdf/ar.ros2_control.xacro" />
   <xacro:include filename="$(find ar_description)/urdf/ar_gripper.ros2_control.xacro" />
-  <xacro:arg name="simulation_controllers" default="" />
+  <!-- clean this up -->
+  <xacro:property name="robot_parameters_file"
+    value="$(find ar_description)/config/$(arg ar_model).yaml" />
+  <xacro:property name="robot_parameters" value="${xacro.load_yaml(robot_parameters_file)}" />
+  <!-- clean this up -->
   <link name="world" />
-  <xacro:ar_robot
-    parent="world"
-    robot_parameters_file="$(find ar_description)/config/$(arg ar_model).yaml"
-  >
-    <origin xyz="0 0 0" rpy="0 0 0" />
-  </xacro:ar_robot>
-  <xacro:ar_gripper parent="ee_link" />
+  <xacro:if value="$(arg include_track)">
+    <xacro:include filename="$(find ar_description)/urdf/ar_track.xacro" />
+    <xacro:ar_track
+      parent="world"
+      robot_parameters_file="$(find ar_description)/config/$(arg ar_model).yaml">
+      <origin xyz="0 0 0" rpy="0 0 0" />
+    </xacro:ar_track>
+    <xacro:ar_robot
+      parent="linear_slider_link"
+      robot_parameters_file="$(find ar_description)/config/$(arg ar_model).yaml">
+      <origin xyz="0 0 ${robot_parameters['linear_plate_height']}" rpy="0 0 0" />
+    </xacro:ar_robot>
+  </xacro:if>
+  <xacro:unless value="$(arg include_track)">
+    <xacro:ar_robot
+      parent="world"
+      robot_parameters_file="$(find ar_description)/config/$(arg ar_model).yaml">
+      <origin xyz="0 0 0" rpy="0 0 0" />
+    </xacro:ar_robot>
+  </xacro:unless>
+  <xacro:if value="$(arg include_gripper)">
+    <xacro:include filename="$(find ar_description)/urdf/ar_gripper_macro.xacro" />
+    <xacro:ar_gripper parent="ee_link" />
+  </xacro:if>
   <xacro:ar_ros2_control
     name="ARGazeboSystem"

File: ar_description/urdf/ar_macro.xacro (robot description, xacro)
@@ -6,29 +6,32 @@
     robot_parameters_file
   ">
-    <xacro:property name="robot_parameters" value="${xacro.load_yaml(robot_parameters_file)}"/>
+    <xacro:property name="robot_parameters" value="${xacro.load_yaml(robot_parameters_file)}" />
     <joint name="base_joint" type="fixed">
       <xacro:insert_block name="origin" />
-      <parent link="${parent}"/>
+      <parent link="${parent}" />
       <child link="base_link" />
     </joint>
     <link name="base_link">
       <inertial>
-        <origin rpy="0 0 0" xyz="-4.6941E-06 0.054174 0.038824"/>
-        <mass value="0.7102"/>
-        <inertia ixx="0.0039943" ixy="3.697E-07" ixz="-5.7364E-08" iyy="0.0014946" iyz="-0.00036051" izz="0.0042554"/>
-      </inertial>
-      <visual>
-        <origin rpy="0 0 0" xyz="0 0 0"/>
-        <geometry>
-          <mesh filename="file://$(find ar_description)/meshes/${robot_parameters['mesh_dir']}/base_link.STL"/>
-        </geometry>
-        <material name="">
-          <color rgba="1 1 0 1"/>
-        </material>
-      </visual>
-      <collision>
-        <origin rpy="0 0 0" xyz="0 0 0"/>
-        <geometry>
-          <mesh filename="file://$(find ar_description)/meshes/${robot_parameters['mesh_dir']}/base_link.STL"/>
+        <origin rpy="0 0 0" xyz="-4.6941E-06 0.054174 0.038824" />
+        <mass value="0.7102" />
+        <inertia ixx="0.0039943" ixy="3.697E-07" ixz="-5.7364E-08" iyy="0.0014946" iyz="-0.00036051"
+          izz="0.0042554" />
+      </inertial>
+      <visual>
+        <origin rpy="0 0 0" xyz="0 0 0" />
+        <geometry>
+          <mesh
+            filename="file://$(find ar_description)/meshes/${robot_parameters['mesh_dir']}/base_link.STL" />
+        </geometry>
+        <material name="">
+          <color rgba="1 1 0 1" />
+        </material>
+      </visual>
+      <collision>
+        <origin rpy="0 0 0" xyz="0 0 0" />
+        <geometry>
+          <mesh
+            filename="file://$(find ar_description)/meshes/${robot_parameters['mesh_dir']}/base_link.STL" />
         </geometry>
       </collision>
@@ -36,175 +39,195 @@
     <link name="link_1">
       <inertial>
-        <origin rpy="0 0 0" xyz="-0.022706 0.04294 -0.12205"/>
-        <mass value="0.88065"/>
-        <inertia ixx="0.0034" ixy="0.00042296" ixz="-0.00089231" iyy="0.0041778" iyz="0.0010848" izz="0.0027077"/>
-      </inertial>
-      <visual>
-        <origin rpy="0 0 0" xyz="0 0 0"/>
-        <geometry>
-          <mesh filename="file://$(find ar_description)/meshes/${robot_parameters['mesh_dir']}/link_1.STL"/>
-        </geometry>
-        <material name="">
-          <color rgba="1 1 0 1"/>
-        </material>
-      </visual>
-      <collision>
-        <origin rpy="0 0 0" xyz="0 0 0"/>
-        <geometry>
-          <mesh filename="file://$(find ar_description)/meshes/${robot_parameters['mesh_dir']}/link_1.STL"/>
+        <origin rpy="0 0 0" xyz="-0.022706 0.04294 -0.12205" />
+        <mass value="0.88065" />
+        <inertia ixx="0.0034" ixy="0.00042296" ixz="-0.00089231" iyy="0.0041778" iyz="0.0010848"
+          izz="0.0027077" />
+      </inertial>
+      <visual>
+        <origin rpy="0 0 0" xyz="0 0 0" />
+        <geometry>
+          <mesh
+            filename="file://$(find ar_description)/meshes/${robot_parameters['mesh_dir']}/link_1.STL" />
+        </geometry>
+        <material name="">
+          <color rgba="1 1 0 1" />
+        </material>
+      </visual>
+      <collision>
+        <origin rpy="0 0 0" xyz="0 0 0" />
+        <geometry>
+          <mesh
+            filename="file://$(find ar_description)/meshes/${robot_parameters['mesh_dir']}/link_1.STL" />
         </geometry>
       </collision>
     </link>
     <joint name="joint_1" type="revolute">
-      <origin rpy="${pi} 0 0" xyz="0 0 0"/>
-      <parent link="base_link"/>
-      <child link="link_1"/>
-      <axis xyz="0 0 1"/>
-      <limit lower="${-170.0 / 180.0 * pi}" upper="${170.0 / 180.0 * pi}" effort="0" velocity="0.5"/>
+      <origin rpy="${pi} 0 0" xyz="0 0 0" />
+      <parent link="base_link" />
+      <child link="link_1" />
+      <axis xyz="0 0 1" />
+      <limit lower="${-170.0 / 180.0 * pi}" upper="${170.0 / 180.0 * pi}" effort="0" velocity="0.5" />
     </joint>
     <link name="link_2">
       <inertial>
-        <origin rpy="0 0 0" xyz="0.064818 -0.11189 -0.038671"/>
-        <mass value="0.57738"/>
-        <inertia ixx="0.0047312" ixy="0.0022624" ixz="0.00032144" iyy="0.0020836" iyz="-0.00056569" izz="0.0056129"/>
-      </inertial>
-      <visual>
-        <origin rpy="0 0 0" xyz="0 0 0"/>
-        <geometry>
-          <mesh filename="file://$(find ar_description)/meshes/${robot_parameters['mesh_dir']}/link_2.STL"/>
-        </geometry>
-        <material name="">
-          <color rgba="1 1 0 1"/>
-        </material>
-      </visual>
-      <collision>
-        <origin rpy="0 0 0" xyz="0 0 0"/>
-        <geometry>
-          <mesh filename="file://$(find ar_description)/meshes/${robot_parameters['mesh_dir']}/link_2.STL"/>
+        <origin rpy="0 0 0" xyz="0.064818 -0.11189 -0.038671" />
+        <mass value="0.57738" />
+        <inertia ixx="0.0047312" ixy="0.0022624" ixz="0.00032144" iyy="0.0020836" iyz="-0.00056569"
+          izz="0.0056129" />
+      </inertial>
+      <visual>
+        <origin rpy="0 0 0" xyz="0 0 0" />
+        <geometry>
+          <mesh
+            filename="file://$(find ar_description)/meshes/${robot_parameters['mesh_dir']}/link_2.STL" />
+        </geometry>
+        <material name="">
+          <color rgba="1 1 0 1" />
+        </material>
+      </visual>
+      <collision>
+        <origin rpy="0 0 0" xyz="0 0 0" />
+        <geometry>
+          <mesh
+            filename="file://$(find ar_description)/meshes/${robot_parameters['mesh_dir']}/link_2.STL" />
         </geometry>
       </collision>
     </link>
     <joint name="joint_2" type="revolute">
-      <origin rpy="1.5708 0 -1.5708" xyz="0 0.0642 -0.16977"/>
-      <parent link="link_1"/>
-      <child link="link_2"/>
-      <axis xyz="0 0 -1"/>
-      <limit lower="${-42.0 / 180.0 * pi}" upper="${90.0 / 180.0 * pi}" effort="0.5" velocity="0.5"/>
+      <origin rpy="1.5708 0 -1.5708" xyz="0 0.0642 -0.16977" />
+      <parent link="link_1" />
+      <child link="link_2" />
+      <axis xyz="0 0 -1" />
+      <limit lower="${-42.0 / 180.0 * pi}" upper="${90.0 / 180.0 * pi}" effort="0.5" velocity="0.5" />
     </joint>
     <link name="link_3">
       <inertial>
-        <origin rpy="0 0 0" xyz="-0.00029765 -0.023661 -0.0019125"/>
-        <mass value="0.1787"/>
-        <inertia ixx="0.0001685" ixy="-2.7713E-05" ixz="5.6885E-06" iyy="0.00012865" iyz="2.9256E-05" izz="0.00020744"/>
-      </inertial>
-      <visual>
-        <origin rpy="0 0 0" xyz="0 0 0"/>
-        <geometry>
-          <mesh filename="file://$(find ar_description)/meshes/${robot_parameters['mesh_dir']}/link_3.STL"/>
-        </geometry>
-        <material name="">
-          <color rgba="1 1 0 1"/>
-        </material>
-      </visual>
-      <collision>
-        <origin rpy="0 0 0" xyz="0 0 0"/>
-        <geometry>
-          <mesh filename="file://$(find ar_description)/meshes/${robot_parameters['mesh_dir']}/link_3.STL"/>
+        <origin rpy="0 0 0" xyz="-0.00029765 -0.023661 -0.0019125" />
+        <mass value="0.1787" />
+        <inertia ixx="0.0001685" ixy="-2.7713E-05" ixz="5.6885E-06" iyy="0.00012865"
+          iyz="2.9256E-05" izz="0.00020744" />
+      </inertial>
+      <visual>
+        <origin rpy="0 0 0" xyz="0 0 0" />
+        <geometry>
+          <mesh
+            filename="file://$(find ar_description)/meshes/${robot_parameters['mesh_dir']}/link_3.STL" />
+        </geometry>
+        <material name="">
+          <color rgba="1 1 0 1" />
+        </material>
+      </visual>
+      <collision>
+        <origin rpy="0 0 0" xyz="0 0 0" />
+        <geometry>
+          <mesh
+            filename="file://$(find ar_description)/meshes/${robot_parameters['mesh_dir']}/link_3.STL" />
         </geometry>
       </collision>
     </link>
     <joint name="joint_3" type="revolute">
-      <origin rpy="0 0 3.1416" xyz="0 -0.305 0.007"/>
-      <parent link="link_2"/>
-      <child link="link_3"/>
-      <axis xyz="0 0 -1"/>
-      <limit lower="${-89.0 / 180.0 * pi}" upper="${52.0 / 180.0 * pi}" effort="0" velocity="0.5"/>
+      <origin rpy="0 0 3.1416" xyz="0 -0.305 0.007" />
+      <parent link="link_2" />
+      <child link="link_3" />
+      <axis xyz="0 0 -1" />
+      <limit lower="${-89.0 / 180.0 * pi}" upper="${52.0 / 180.0 * pi}" effort="0" velocity="0.5" />
     </joint>
     <link name="link_4">
       <inertial>
-        <origin rpy="0 0 0" xyz="-0.0016798 -0.00057319 -0.074404"/>
-        <mass value="0.34936"/>
-        <inertia ixx="0.0030532" ixy="-1.8615E-05" ixz="-7.0047E-05" iyy="0.0031033" iyz="-2.3301E-05" izz="0.00022264"/>
-      </inertial>
-      <visual>
-        <origin rpy="0 0 0" xyz="0 0 0"/>
-        <geometry>
-          <mesh filename="file://$(find ar_description)/meshes/${robot_parameters['mesh_dir']}/link_4.STL"/>
-        </geometry>
-        <material name="">
-          <color rgba="1 1 0 1"/>
-        </material>
-      </visual>
-      <collision>
-        <origin rpy="0 0 0" xyz="0 0 0"/>
-        <geometry>
-          <mesh filename="file://$(find ar_description)/meshes/${robot_parameters['mesh_dir']}/link_4.STL"/>
+        <origin rpy="0 0 0" xyz="-0.0016798 -0.00057319 -0.074404" />
+        <mass value="0.34936" />
+        <inertia ixx="0.0030532" ixy="-1.8615E-05" ixz="-7.0047E-05" iyy="0.0031033"
+          iyz="-2.3301E-05" izz="0.00022264" />
+      </inertial>
+      <visual>
+        <origin rpy="0 0 0" xyz="0 0 0" />
+        <geometry>
+          <mesh
+            filename="file://$(find ar_description)/meshes/${robot_parameters['mesh_dir']}/link_4.STL" />
+        </geometry>
+        <material name="">
+          <color rgba="1 1 0 1" />
+        </material>
+      </visual>
+      <collision>
+        <origin rpy="0 0 0" xyz="0 0 0" />
+        <geometry>
+          <mesh
+            filename="file://$(find ar_description)/meshes/${robot_parameters['mesh_dir']}/link_4.STL" />
         </geometry>
       </collision>
     </link>
     <joint name="joint_4" type="revolute">
-      <origin rpy="1.5708 0 -1.5708" xyz="0 0 0.0"/>
-      <parent link="link_3"/>
-      <child link="link_4"/>
-      <axis xyz="0 0 -1"/>
-      <limit lower="${-1 * robot_parameters['j4_limit']}" upper="${robot_parameters['j4_limit']}" effort="0" velocity="0.5"/>
+      <origin rpy="1.5708 0 -1.5708" xyz="0 0 0.0" />
+      <parent link="link_3" />
+      <child link="link_4" />
+      <axis xyz="0 0 -1" />
+      <limit lower="${-1 * robot_parameters['j4_limit']}" upper="${robot_parameters['j4_limit']}"
+        effort="0" velocity="0.5" />
     </joint>
     <link name="link_5">
       <inertial>
-        <origin rpy="0 0 0" xyz="0.0015066 -1.3102E-05 -0.012585"/>
-        <mass value="0.11562"/>
-        <inertia ixx="5.5035E-05" ixy="-1.019E-08" ixz="-2.6243E-06" iyy="8.2921E-05" iyz="1.4437E-08" izz="5.2518E-05"/>
-      </inertial>
-      <visual>
-        <origin rpy="0 0 0" xyz="0 0 0"/>
-        <geometry>
-          <mesh filename="file://$(find ar_description)/meshes/${robot_parameters['mesh_dir']}/link_5.STL"/>
-        </geometry>
-        <material name="">
-          <color rgba="1 1 0 1"/>
-        </material>
-      </visual>
-      <collision>
-        <origin rpy="0 0 0" xyz="0 0 0"/>
-        <geometry>
-          <mesh filename="file://$(find ar_description)/meshes/${robot_parameters['mesh_dir']}/link_5.STL"/>
+        <origin rpy="0 0 0" xyz="0.0015066 -1.3102E-05 -0.012585" />
+        <mass value="0.11562" />
+        <inertia ixx="5.5035E-05" ixy="-1.019E-08" ixz="-2.6243E-06" iyy="8.2921E-05"
+          iyz="1.4437E-08" izz="5.2518E-05" />
+      </inertial>
+      <visual>
+        <origin rpy="0 0 0" xyz="0 0 0" />
+        <geometry>
+          <mesh
+            filename="file://$(find ar_description)/meshes/${robot_parameters['mesh_dir']}/link_5.STL" />
+        </geometry>
+        <material name="">
+          <color rgba="1 1 0 1" />
+        </material>
+      </visual>
+      <collision>
+        <origin rpy="0 0 0" xyz="0 0 0" />
+        <geometry>
+          <mesh
+            filename="file://$(find ar_description)/meshes/${robot_parameters['mesh_dir']}/link_5.STL" />
         </geometry>
       </collision>
     </link>
     <joint name="joint_5" type="revolute">
-      <origin rpy="${pi} 0 -1.5708" xyz="0 0 -0.22263"/>
-      <parent link="link_4"/>
-      <child link="link_5"/>
-      <axis xyz="1 0 0"/>
-      <limit lower="${-105.0 / 180.0 * pi}" upper="${105.0 / 180.0 * pi}" effort="0" velocity="1.0"/>
+      <origin rpy="${pi} 0 -1.5708" xyz="0 0 -0.22263" />
+      <parent link="link_4" />
+      <child link="link_5" />
+      <axis xyz="1 0 0" />
+      <limit lower="${-105.0 / 180.0 * pi}" upper="${105.0 / 180.0 * pi}" effort="0" velocity="1.0" />
     </joint>
     <link name="link_6">
       <inertial>
-        <origin rpy="0 0 0" xyz="2.9287E-10 -1.6472E-09 0.0091432"/>
-        <mass value="0.013863"/>
-        <inertia ixx="1.3596E-06" ixy="3.0585E-13" ixz="5.7102E-14" iyy="1.7157E-06" iyz="6.3369E-09" izz="2.4332E-06"/>
-      </inertial>
-      <visual>
-        <origin rpy="0 0 0" xyz="0 0 0"/>
-        <geometry>
-          <mesh filename="file://$(find ar_description)/meshes/${robot_parameters['mesh_dir']}/link_6.STL"/>
-        </geometry>
-        <material name="">
-          <color rgba="1 1 0 1"/>
-        </material>
-      </visual>
-      <collision>
-        <origin rpy="0 0 0" xyz="0 0 0"/>
-        <geometry>
-          <mesh filename="file://$(find ar_description)/meshes/${robot_parameters['mesh_dir']}/link_6.STL"/>
+        <origin rpy="0 0 0" xyz="2.9287E-10 -1.6472E-09 0.0091432" />
+        <mass value="0.013863" />
+        <inertia ixx="1.3596E-06" ixy="3.0585E-13" ixz="5.7102E-14" iyy="1.7157E-06"
+          iyz="6.3369E-09" izz="2.4332E-06" />
+      </inertial>
+      <visual>
+        <origin rpy="0 0 0" xyz="0 0 0" />
+        <geometry>
+          <mesh
+            filename="file://$(find ar_description)/meshes/${robot_parameters['mesh_dir']}/link_6.STL" />
+        </geometry>
+        <material name="">
+          <color rgba="1 1 0 1" />
+        </material>
+      </visual>
+      <collision>
+        <origin rpy="0 0 0" xyz="0 0 0" />
+        <geometry>
+          <mesh
+            filename="file://$(find ar_description)/meshes/${robot_parameters['mesh_dir']}/link_6.STL" />
         </geometry>
       </collision>
     </link>
     <joint name="joint_6" type="revolute">
-      <origin rpy="0 0 3.1416" xyz="0.000 0 ${robot_parameters['l6_length']}"/>
-      <parent link="link_5"/>
-      <child link="link_6"/>
-      <axis xyz="0 0 1"/>
-      <limit lower="${-1.0 * robot_parameters['j6_limit']}" upper="${robot_parameters['j6_limit']}" effort="0" velocity="1.0"/>
+      <origin rpy="0 0 3.1416" xyz="0.000 0 ${robot_parameters['l6_length']}" />
+      <parent link="link_5" />
+      <child link="link_6" />
+      <axis xyz="0 0 1" />
+      <limit lower="${-1.0 * robot_parameters['j6_limit']}" upper="${robot_parameters['j6_limit']}"
+        effort="0" velocity="1.0" />
     </joint>
     <!-- center of the end effector mounting surface on link_6 -->

File: ar_moveit_config/srdf/ar.srdf.xacro (robot description, xacro)
@@ -1,9 +1,14 @@
 <?xml version="1.0" encoding="UTF-8"?>
 <robot xmlns:xacro="http://wiki.ros.org/xacro" name="$(arg name)">
-  <xacro:arg name="include_gripper" default="true"/>
-  <xacro:include filename="$(find ar_moveit_config)/srdf/ar_macro.srdf.xacro"/>
+  <xacro:arg name="include_gripper" default="true" />
+  <xacro:arg name="include_track" default="true" />
+  <xacro:if value="$(arg include_track)">
+    <xacro:include filename="$(find ar_moveit_config)/srdf/ar_track_macro.srdf.xacro" />
+    <xacro:ar_track_srdf />
+  </xacro:if>
+  <xacro:include filename="$(find ar_moveit_config)/srdf/ar_macro.srdf.xacro" />
   <xacro:ar_srdf />
   <xacro:if value="$(arg include_gripper)">
-    <xacro:include filename="$(find ar_moveit_config)/srdf/ar_gripper_macro.srdf.xacro"/>
+    <xacro:include filename="$(find ar_moveit_config)/srdf/ar_gripper_macro.srdf.xacro" />
     <xacro:ar_gripper_srdf />
   </xacro:if>

File: ar_moveit_config/srdf/ar_macro.srdf.xacro (robot description, xacro)
@@ -2,5 +2,6 @@
 <!--This does not replace URDF, and is not an extension of URDF.
     This is a format for representing semantic information about the robot structure.
-    A URDF file must exist for this robot as well, where the joints and the links that are referenced are defined
+    A URDF file must exist for this robot as well, where the joints and the links that are referenced
+are defined
 -->
 <robot xmlns:xacro="http://wiki.ros.org/xacro">
