Commit message: Trying to make 6 dof work w/ inc_track=false

File: ar_description/urdf/ar.ros2_control.xacro (robot description, xacro)
@@ -9,6 +9,10 @@
     joint_offset_parameters_file
   ">
+    <xacro:arg name="include_track" default="True" />
     <xacro:property name="joint_offset_parameters"
       value="${xacro.load_yaml(joint_offset_parameters_file)}" />
+    <xacro:property name="robot_parameters_file"
+      value="$(find ar_description)/config/$(arg ar_model).yaml" />
+    <xacro:property name="robot_parameters" value="${xacro.load_yaml(robot_parameters_file)}" />
     <ros2_control name="${name}" type="system">
       <hardware>
@@ -17,14 +21,16 @@
         <param name="calibrate">${calibrate}</param>
       </hardware>
-      <joint name="linear_slider_joint">
-        <command_interface name="position">
-          <param name="min">{-0.6/2+0.15/2}</param>
-          <param name="max">{0.6/2-0.15/2}</param>
-        </command_interface>
-        <state_interface name="position">
-          <param name="initial_value">0.0</param>
-        </state_interface>
-        <param name="position_offset">${joint_offset_parameters['linear_track']}</param>
-      </joint>
+      <xacro:if value="$(arg include_track)">
+        <joint name="linear_slider_joint">
+          <command_interface name="position">
+            <param name="min">${-robot_parameters['linear_track_length']/2+0.15/2}</param>
+            <param name="max">${robot_parameters['linear_track_length']/2-0.15/2}</param>
+          </command_interface>
+          <state_interface name="position">
+            <param name="initial_value">0.0</param>
+          </state_interface>
+          <param name="position_offset">${joint_offset_parameters['linear_track']}</param>
+        </joint>
+      </xacro:if>
       <joint name="joint_1">
         <command_interface name="position">

File: ar_description/urdf/ar_track_macro.xacro (robot description, xacro)
@@ -20,5 +20,5 @@
         <geometry>
           <box
-            size="${robot_parameters['linear_track_length']} 0.3 ${robot_parameters['linear_track_height']}" />
+            size="${robot_parameters['linear_track_length']} ${robot_parameters['linear_track_width']} ${robot_parameters['linear_track_height']}" />
         </geometry>
         <material name="">
@@ -30,5 +30,5 @@
         <geometry>
           <box
-            size="${robot_parameters['linear_track_length']} 0.3 ${robot_parameters['linear_track_height']}" />
+            size="${robot_parameters['linear_track_length']} ${robot_parameters['linear_track_width']} ${robot_parameters['linear_track_height']}" />
         </geometry>
       </collision>
@@ -39,6 +39,8 @@
       <origin xyz="0 0 ${robot_parameters['linear_track_height']}" rpy="0 0 0" />
       <axis xyz="1 0 0" />
-      <limit lower="${-robot_parameters['linear_track_length']/2+0.15/2}"
-        upper="${robot_parameters['linear_track_length']/2-0.15/2}" effort="100" velocity="0.5" />
+      <limit
+        lower="${-(robot_parameters['linear_track_length']+robot_parameters['linear_track_width']) /2}"
+        upper="${(robot_parameters['linear_track_length']-robot_parameters['linear_track_width']) /2}"
+        effort="100" velocity="0.5" />
     </joint>
     <link name="linear_slider_link">
@@ -51,5 +53,6 @@
         <origin xyz="0 0 ${robot_parameters['linear_plate_height'] / 2}" rpy="0 0 0" />
         <geometry>
-          <box size="0.15 0.3 ${robot_parameters['linear_plate_height']}" />
+          <box
+            size="${robot_parameters['linear_plate_width']} ${robot_parameters['linear_plate_length']} ${robot_parameters['linear_plate_height']}" />
         </geometry>
         <material name="">
@@ -60,5 +63,6 @@
         <origin xyz="0 0 ${robot_parameters['linear_plate_height'] / 2}" rpy="0 0 0" />
         <geometry>
-          <box size="0.15 0.3 ${robot_parameters['linear_plate_height']}" />
+          <box
+            size="${robot_parameters['linear_plate_width']} ${robot_parameters['linear_plate_length']} ${robot_parameters['linear_plate_height']}" />
         </geometry>
       </collision>

Commit message: Track graphics, cleaned up urdf

File: ar_description/urdf/ar.ros2_control.xacro (robot description, xacro)
@@ -24,6 +24,8 @@
         <joint name="linear_slider_joint">
           <command_interface name="position">
-            <param name="min">${-robot_parameters['linear_track_length']/2+0.15/2}</param>
-            <param name="max">${robot_parameters['linear_track_length']/2-0.15/2}</param>
+            <param name="min">
+              ${-(robot_parameters['linear_track_length']+robot_parameters['linear_plate_width'])/2}</param>
+            <param name="max">
+              ${(robot_parameters['linear_track_length']-robot_parameters['linear_plate_width'])/2}</param>
           </command_interface>
           <state_interface name="position">

File: ar_description/urdf/ar_gazebo.urdf.xacro (robot description, xacro)
@@ -10,5 +10,5 @@
     value="$(find ar_description)/config/$(arg ar_model).yaml" />
   <xacro:property name="robot_parameters" value="${xacro.load_yaml(robot_parameters_file)}" />
-  <link name="world" />
+  <link name="world" /> <!-- rename to have robot "free"-->
   <xacro:property name="ar_robot_parent" value="world" />
   <xacro:property name="ar_robot_origin_xyz" value="0 0 0" />

File: ar_description/urdf/ar_track_macro.xacro (robot description, xacro)
@@ -5,4 +5,10 @@
   robot_parameters_file">
     <xacro:property name="robot_parameters" value="${xacro.load_yaml(robot_parameters_file)}" />
+    <xacro:property name="plate_width" value="${robot_parameters['linear_plate_width']}" />
+    <xacro:property name="plate_length" value="${robot_parameters['linear_plate_length']}" />
+    <xacro:property name="plate_height" value="${robot_parameters['linear_plate_height']}" />
+    <xacro:property name="track_width" value="${robot_parameters['linear_track_width']}" />
+    <xacro:property name="track_length" value="${robot_parameters['linear_track_length']}" />
+    <xacro:property name="track_height" value="${robot_parameters['linear_track_height']}" />
     <joint name="linear_base_joint" type="fixed">
       <xacro:insert_block name="origin" />
@@ -17,8 +23,22 @@
       </inertial>
       <visual>
-        <origin xyz="0 0 ${robot_parameters['linear_track_height'] / 2}" rpy="0 0 0" />
+        <origin
+          xyz="0 ${-track_width/2+0.03/2} ${track_height / 2}"
+          rpy="0 0 0" />
         <geometry>
-          <box
-            size="${robot_parameters['linear_track_length']} ${robot_parameters['linear_track_width']} ${robot_parameters['linear_track_height']}" />
+          <mesh
+            filename="file://$(find ar_description)/meshes/${robot_parameters['mesh_dir']}/track.stl" />
+        </geometry>
+        <material name="">
+          <color rgba="1 1 0 1" />
+        </material>
+      </visual>
+      <visual>
+        <origin
+          xyz="0 ${track_width/2-0.03/2} ${track_height / 2}"
+          rpy="0 0 0" />
+        <geometry>
+          <mesh
+            filename="file://$(find ar_description)/meshes/${robot_parameters['mesh_dir']}/track.stl" />
         </geometry>
         <material name="">
@@ -27,8 +47,8 @@
       </visual>
       <collision>
-        <origin xyz="0 0 ${robot_parameters['linear_track_height'] / 2}" rpy="0 0 0" />
+        <origin xyz="0 0 ${track_height / 2}" rpy="0 0 0" />
         <geometry>
           <box
-            size="${robot_parameters['linear_track_length']} ${robot_parameters['linear_track_width']} ${robot_parameters['linear_track_height']}" />
+            size="${track_length} ${track_width} ${track_height}" />
         </geometry>
       </collision>
@@ -37,9 +57,9 @@
       <parent link="linear_base_link" />
       <child link="linear_slider_link" />
-      <origin xyz="0 0 ${robot_parameters['linear_track_height']}" rpy="0 0 0" />
+      <origin xyz="0 0 ${track_height}" rpy="0 0 0" />
       <axis xyz="1 0 0" />
       <limit
-        lower="${-(robot_parameters['linear_track_length']+robot_parameters['linear_track_width']) /2}"
-        upper="${(robot_parameters['linear_track_length']-robot_parameters['linear_track_width']) /2}"
+        lower="${(-track_length+plate_width) /2}"
+        upper="${(track_length-plate_width) /2}"
         effort="100" velocity="0.5" />
     </joint>
@@ -51,8 +71,20 @@
       </inertial>
       <visual>
-        <origin xyz="0 0 ${robot_parameters['linear_plate_height'] / 2}" rpy="0 0 0" />
+        <origin xyz="0 0 ${plate_height / 2}" rpy="0 0 0" />
         <geometry>
           <box
-            size="${robot_parameters['linear_plate_width']} ${robot_parameters['linear_plate_length']} ${robot_parameters['linear_plate_height']}" />
+            size="${plate_width} ${plate_length} ${plate_height}" />
+        </geometry>
+        <material name="">
+          <color rgba="1 1 0 1" />
+        </material>
+      </visual>
+      <visual>
+        <origin
+          xyz="${plate_width/2} ${plate_length/2} ${-plate_height / 2}"
+          rpy="0 0 0" />
+        <geometry>
+          <mesh
+            filename="file://$(find ar_description)/meshes/${robot_parameters['mesh_dir']}/track_bearing.stl" />
         </geometry>
         <material name="">
@@ -61,8 +93,8 @@
       </visual>
       <collision>
-        <origin xyz="0 0 ${robot_parameters['linear_plate_height'] / 2}" rpy="0 0 0" />
+        <origin xyz="0 0 ${plate_height / 2}" rpy="0 0 0" />
         <geometry>
           <box
-            size="${robot_parameters['linear_plate_width']} ${robot_parameters['linear_plate_length']} ${robot_parameters['linear_plate_height']}" />
+            size="${plate_width} ${plate_length} ${plate_height}" />
         </geometry>
       </collision>

Commit message: FINALLY BRILLIANT

File: ar_description/urdf/ar.ros2_control.xacro (robot description, xacro)
@@ -21,18 +21,4 @@
         <param name="calibrate">${calibrate}</param>
       </hardware>
-      <xacro:if value="$(arg include_track)">
-        <joint name="linear_slider_joint">
-          <command_interface name="position">
-            <param name="min">
-              ${-(robot_parameters['linear_track_length']+robot_parameters['linear_plate_width'])/2}</param>
-            <param name="max">
-              ${(robot_parameters['linear_track_length']-robot_parameters['linear_plate_width'])/2}</param>
-          </command_interface>
-          <state_interface name="position">
-            <param name="initial_value">0.0</param>
-          </state_interface>
-          <param name="position_offset">${joint_offset_parameters['linear_track']}</param>
-        </joint>
-      </xacro:if>
       <joint name="joint_1">
         <command_interface name="position">
@@ -95,4 +81,18 @@
         <param name="position_offset">${joint_offset_parameters['joint_6']}</param>
       </joint>
+      <xacro:if value="$(arg include_track)">
+        <joint name="linear_slider_joint">
+          <command_interface name="position">
+            <param name="min">
+              ${-(robot_parameters['linear_track_length']+robot_parameters['linear_plate_width'])/2}</param>
+            <param name="max">
+              ${(robot_parameters['linear_track_length']-robot_parameters['linear_plate_width'])/2}</param>
+          </command_interface>
+          <state_interface name="position">
+            <param name="initial_value">0.0</param>
+          </state_interface>
+          <param name="position_offset">${joint_offset_parameters['linear_track']}</param>
+        </joint>
+      </xacro:if>
     </ros2_control>
   </xacro:macro>

File: ar_description/urdf/ar_track_macro.xacro (robot description, xacro)
@@ -89,5 +89,5 @@
       <limit
         lower="${(-track_length+plate_width) /2}"
-        upper="${(track_length-plate_width) /2}"
+        upper="${(track_length-plate_width)/2}"
         effort="100" velocity="0.5" />
     </joint>

File: ar_moveit_config/srdf/ar.srdf.xacro (robot description, xacro)
@@ -3,8 +3,4 @@
   <xacro:arg name="include_gripper" default="True" />
   <xacro:arg name="include_track" default="True" />
-  <xacro:if value="$(arg include_track)">
-    <xacro:include filename="$(find ar_moveit_config)/srdf/ar_track_macro.srdf.xacro" />
-    <xacro:ar_track_srdf />
-  </xacro:if>
   <xacro:include filename="$(find ar_moveit_config)/srdf/ar_macro.srdf.xacro" />
   <xacro:ar_srdf />

File: ar_moveit_config/srdf/ar_macro.srdf.xacro (robot description, xacro)
@@ -54,4 +54,8 @@
       <joint name="joint_6" value="0" />
     </group_state>
+    <xacro:if value="$(arg include_track)">
+      <disable_collisions link1="linear_base_link" link2="linear_slider_link" reason="Adjacent" />
+      <disable_collisions link1="linear_slider_link" link2="base_link" reason="Adjacent" />
+    </xacro:if>
     <disable_collisions link1="base_link" link2="link_1" reason="Adjacent" />
     <disable_collisions link1="link_1" link2="link_2" reason="Adjacent" />
