Commit message: demo is up again!

File: ar_moveit_config/urdf/fake_ar.urdf.xacro (robot description, xacro)
@@ -5,12 +5,33 @@
   <xacro:include filename="$(find ar_description)/urdf/ar.ros2_control.xacro" />
   <xacro:include filename="$(find ar_description)/urdf/ar_gripper.ros2_control.xacro" />
+  <xacro:arg name="include_gripper" default="True" />
+  <xacro:arg name="include_track" default="True" />
+  <xacro:include filename="$(find ar_description)/urdf/ar_macro.xacro" />
+  <xacro:property name="robot_parameters_file"
+    value="$(find ar_description)/config/$(arg ar_model).yaml" />
+  <xacro:property name="robot_parameters" value="${xacro.load_yaml(robot_parameters_file)}" />
   <link name="world" />
+  <xacro:property name="ar_robot_parent" value="world" />
+  <xacro:property name="ar_robot_origin_xyz" value="0 0 0" />
+  <xacro:if value="$(arg include_track)">
+    <xacro:include filename="$(find ar_description)/urdf/ar_track_macro.xacro" />
+    <xacro:ar_track
+      parent="world"
+      robot_parameters_file="${robot_parameters_file}">
+      <origin xyz="0 0 0" rpy="0 0 0" />
+    </xacro:ar_track>
+    <xacro:property name="ar_robot_parent" value="linear_slider_link" />
+    <xacro:property name="ar_robot_origin_xyz"
+      value="0 0 ${robot_parameters['linear_plate_height']}" />
+  </xacro:if>
   <xacro:ar_robot
-    parent="world"
-    robot_parameters_file="$(find ar_description)/config/$(arg ar_model).yaml"
-  >
-    <origin xyz="0 0 0" rpy="0 0 0" />
+    parent="${ar_robot_parent}"
+    robot_parameters_file="${robot_parameters_file}">
+    <origin xyz="${ar_robot_origin_xyz}" rpy="0 0 0" />
   </xacro:ar_robot>
-  <xacro:ar_gripper parent="ee_link" />
+  <xacro:if value="$(arg include_gripper)">
+    <xacro:include filename="$(find ar_description)/urdf/ar_gripper_macro.xacro" />
+    <xacro:ar_gripper parent="ee_link" />
+  </xacro:if>
   <xacro:ar_ros2_control
     name="ARFakeSystem"
